File: Elec_Schematic/OSDWatch/OSDWatch.sch (KiCad schematic (older format))
At the start: 4 parts, among them U1 ESP32DEVKITV1, U2 ADXL345_Module, U3 MAX30102_Module, U4 OLED_Display

Commit message: Added notifications between tasks and main app so we let one task initialise before starting the next one - therwise I2C bus got in a tizz.
Parts:
- added D1: LED, symbol Device:LED
- added R1: 10k0, symbol Device:R_Small
Connections:
- net at U1.2 (GND), U2.1 (GND), U3.GND (7)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: now also R1.2
- net at U1.3 (D15): now also D1.2 (A)
- new net: D1.1 (K), R1.1
Changed lines of the file:
@@
 	4700 4050 4250 4050
-Wire Wire Line
-	1800 4050 1800 2500
 Wire Wire Line
 	4700 4750 4250 4750
@@
 Wire Wire Line
 	1900 800  1900 1100
+$Comp
+L Device:LED D1
+U 1 1 5C0BB649
+P 2150 2800
+F 0 "D1" V 2188 2683 50  0000 R CNN
+F 1 "LED" V 2097 2683 50  0000 R CNN
+F 2 "" H 2150 2800 50  0001 C CNN
+F 3 "~" H 2150 2800 50  0001 C CNN
+	1    2150 2800
+	0    -1   -1   0
+$EndComp
+Wire Wire Line
+	1900 2500 1900 2650
+Wire Wire Line
+	1800 2500 1800 3000
+$Comp
+L Device:R_Small R1
+U 1 1 5C0BE3DC
+P 1950 3000
+F 0 "R1" V 1754 3000 50  0000 C CNN
+F 1 "10k0" V 1845 3000 50  0000 C CNN
+F 2 "" H 1950 3000 50  0001 C CNN
+F 3 "~" H 1950 3000 50  0001 C CNN
+	1    1950 3000
+	0    1    1    0
+$EndComp
+Wire Wire Line
+	1900 2650 2150 2650
+Wire Wire Line
+	2150 2950 2150 3000
+Wire Wire Line
+	2150 3000 2050 3000
+Wire Wire Line
+	1850 3000 1800 3000
+Connection ~ 1800 3000
+Wire Wire Line
+	1800 3000 1800 4050
 $EndSCHEMATC
